File: L298-Breakout_s.sch (EAGLE design)
At the start: 2 parts, among them U1 L298

Commit message: Added web address
Other:
- note added: "By Eason Smith"
- note added: "www.EasonRobotics.com"
- note removed: "Eason Smith"
Changed lines of the file:
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@@
 <sheet>
 <plain>
-<text x="123.19" y="5.334" size="2.54" layer="94" font="vector">Eason Smith</text>
+<text x="123.19" y="5.334" size="2.54" layer="94" font="vector">By Eason Smith</text>
 <text x="96.52" y="93.98" size="1.778" layer="94" font="vector">REV: 8-30-14</text>
 <text x="35.56" y="101.6" size="5.08" layer="94">L298 Breakout Board v1.0</text>
@@
 <wire x1="119.38" y1="109.22" x2="33.02" y2="109.22" width="0.8128" layer="94"/>
 <wire x1="33.02" y1="109.22" x2="33.02" y2="99.06" width="0.8128" layer="94"/>
+<text x="71.12" y="-2.54" size="2.54" layer="94" font="vector">www.EasonRobotics.com</text>
 </plain>
 <instances>
